File: BAGS/Eagle/Container/Cansat2019_1516_Container_v01.brd (EAGLE design)
At the start: 160 x 100 mm, 32 parts, among them IC1 LM1117-3.3V-SOT223, IC2 24C64SM, Q1 MOSFET-NCHANNEL2N7000, Q2 TIP120, U1 TINY45-20-DIP

Commit message: Add files via upload
Parts:
- removed U$1: MT3608_BOB, Breakouts:MT3608_BOB
- added MT3608: MT3608_BOB, Breakouts:MT3608_BOB
- added SWITCH: (no value), CEDT_JANUARY_2015_v5:02P
- moved C3 134.2 mm to (52.1, 7.62), turned to 180 degrees
- moved NICH_LED 126.5 mm to (58.4, 35.6), turned to 90 degrees
- moved PWR_LED 121.5 mm to (67.3, 2.54)
- moved R1 120.7 mm to (59.7, 2.54), turned to 180 degrees
- moved C2 118.4 mm to (52.1, 17.1), turned to 180 degrees
- moved C1 117.0 mm to (52.1, 3.17), turned to 180 degrees
- moved R3 113.7 mm to (52.1, 35.6), turned to 90 degrees
- moved R7 105.7 mm to (54.6, 35.6), turned to 270 degrees
- moved IC2 90.8 mm to (26.7, 20.3), turned to 270 degrees
- moved C4 89.1 mm to (52.1, 12.7), turned to 180 degrees
- moved R5 85.9 mm to (49.5, 35.6)
- moved R6 85.9 mm to (47.0, 35.6)
- moved PROG/DEPL 85.6 mm to (33.0, 44.5)
- moved C5 84.5 mm to (35.6, 40.6)
- moved MCU_LEFT 84.5 mm to (27.9, 33.0)
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Connections:
- new net N$6: BAT_CON.1, SWITCH.2
- net +12V: now also MT3608.VOUT+; no longer U$1.VOUT+
- net GND: now also MT3608.VIN-, MT3608.VOUT-; no longer U$1.VIN-, U$1.VOUT-
- net VBAT: now also MT3608.VIN+, SWITCH.1; no longer BAT_CON.1, U$1.VIN+
Routing:
- net VCC: track 0.00 -> 119.3 mm
- net VBAT: track 0.00 -> 98.7 mm
- net SDA: track 0.00 -> 89.1 mm
- net SCL: track 0.00 -> 77.7 mm, vias 0 -> 1
- net NCH_WIR: track 0.00 -> 38.6 mm
- net BUZZER: track 0.00 -> 37.5 mm
- net RESET: track 0.00 -> 35.0 mm
- net GND: track 0.00 -> 25.7 mm, vias 0 -> 3
- net MISO: track 0.00 -> 24.6 mm
- net N$1: track 0.00 -> 22.1 mm
- net N$2: track 0.00 -> 22.0 mm
- net +12V: track 0.00 -> 14.0 mm
- net MCU_VCC: track 0.00 -> 13.1 mm
- net VPROG: track 0.00 -> 11.5 mm
- net N$5: track 0.00 -> 6.71 mm
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- added copper zone on layer 16, net GND
- added copper zone on layer 1, net VCC
Other:
- board size 160 x 100 mm -> 76.2 x 47.9 mm
