File: BAGS/Eagle/Container/Cansat2019_1516_Container_v01.sch (EAGLE design)
At the start: 27 parts, among them IC1 LM1117-3.3V-SOT223, IC2 24C64SM, Q1 MOSFET-NCHANNEL2N7000, Q2 TIP120, U1 TINY45-20-DIP

Commit message: Add files via upload
Parts:
- added BAT_CON: (no value), CEDT_JANUARY_2015_v5:M02
- added NICH_LED: (no value), 01_adafruit:LED3MM
- added PWR: M04X2, SparkFun-Connectors:M04X2
- added R7: 1k, rcl:R-EU_0204/7
- added U$1: MT3608_BOB, Breakouts:MT3608_BOB
- MCU_LEFT, MCU_RIGHT: device SparkFun-Connectors:M04PTH -> con-amp-quick:M04
Connections:
- new net N$5: NICH_LED.A, R7.1
- net +12V: now also U$1.VOUT+
- net GND: now also BAT_CON.2, NICH_LED.C, PWR.2, PWR.4, PWR.6, PWR.8, U$1.VIN-, U$1.VOUT-
- net NCH_WIR: now also R7.2
- net VBAT: now also BAT_CON.1, PWR.1, PWR.3, PWR.5, PWR.7, U$1.VIN+
Other:
- note removed: "(TODO: 12V Boost circuit)"
- note removed: "(TODO: Add battery connector)"
- moved on the sheet: C1, C2, C3, C4, IC1, NICHROME_WIRE-1, NICHROME_WIRE-2, PWR_LED, Q2, R1, R3

Commit message: Add files via upload
Parts:
- added SWITCH: (no value), CEDT_JANUARY_2015_v5:M02
- renumbered U$1 to MT3608
Connections:
- new net N$6: BAT_CON.1, SWITCH.2
- net VBAT: now also SWITCH.1; no longer BAT_CON.1
Other:
- moved on the sheet: BAT_CON
Changed lines of the file:
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@@
 </variantdefs>
 <classes>
-<class number="0" name="default" width="0" drill="0">
+<class number="0" name="default" width="0.3048" drill="0">
+<clearance class="0" value="0.3048"/>
+</class>
+<class number="1" name="power" width="0.6096" drill="0">
+<clearance class="1" value="0.3048"/>
+</class>
+<class number="2" name="burner" width="0.8128" drill="0">
+<clearance class="2" value="0.3048"/>
 </class>
 </classes>
@@
 <part name="R7" library="rcl" deviceset="R-EU_" device="0204/7" value="1k"/>
 <part name="NICH_LED" library="01_adafruit" deviceset="LED" device="3MM"/>
-<part name="U$1" library="Breakouts" deviceset="MT3608_BOB" device=""/>
+<part name="MT3608" library="Breakouts" deviceset="MT3608_BOB" device=""/>
 <part name="GND8" library="MSP PROJECT LIBRARY" deviceset="GND" device=""/>
 <part name="P+8" library="supply1" deviceset="+12V" device=""/>
@@
 <part name="BAT_CON" library="CEDT_JANUARY_2015_v5" deviceset="M02" device=""/>
 <part name="GND9" library="MSP PROJECT LIBRARY" deviceset="GND" device=""/>
+<part name="SWITCH" library="CEDT_JANUARY_2015_v5" deviceset="M02" device=""/>
 </parts>
 <sheets>
@@
 <instance part="R7" gate="G$1" x="210.82" y="27.94" rot="R180"/>
 <instance part="NICH_LED" gate="G$1" x="223.52" y="27.94" rot="R90"/>
-<instance part="U$1" gate="G$1" x="55.88" y="5.08"/>
+<instance part="MT3608" gate="G$1" x="55.88" y="5.08"/>
 <instance part="GND8" gate="1" x="68.58" y="-20.32"/>
 <instance part="P+8" gate="1" x="96.52" y="7.62"/>
 <instance part="PWR" gate="G$1" x="17.78" y="-5.08"/>
-<instance part="BAT_CON" gate="G$1" x="12.7" y="48.26" rot="MR180"/>
+<instance part="BAT_CON" gate="G$1" x="12.7" y="40.64" rot="MR180"/>
 <instance part="GND9" gate="1" x="27.94" y="-15.24"/>
+<instance part="SWITCH" gate="G$1" x="12.7" y="53.34" rot="MR180"/>
 </instances>
 <busses>
 </busses>
 <nets>
-<net name="VBAT" class="0">
+<net name="VBAT" class="2">
 <segment>
 <pinref part="IC1" gate="G$1" pin="VIN"/>
@@
 <junction x="43.18" y="55.88"/>
 <label x="35.56" y="58.42" size="1.778" layer="95"/>
-<pinref part="BAT_CON" gate="G$1" pin="1"/>
-<wire x1="20.32" y1="48.26" x2="22.86" y2="48.26" width="0.1524" layer="91"/>
-<wire x1="22.86" y1="48.26" x2="22.86" y2="55.88" width="0.1524" layer="91"/>
+<pinref part="SWITCH" gate="G$1" pin="1"/>
+<wire x1="20.32" y1="53.34" x2="22.86" y2="53.34" width="0.1524" layer="91"/>
+<wire x1="22.86" y1="53.34" x2="22.86" y2="55.88" width="0.1524" layer="91"/>
 </segment>
 <segment>
@@
 </segment>
 <segment>
-<pinref part="U$1" gate="G$1" pin="VIN+"/>
+<pinref part="MT3608" gate="G$1" pin="VIN+"/>
 <wire x1="50.8" y1="0" x2="33.02" y2="0" width="0.1524" layer="91"/>
 <label x="33.02" y="0" size="1.778" layer="95"/>
@@
 </segment>
 </net>
-<net name="VCC" class="0">
+<net name="VCC" class="1">
 <segment>
 <pinref part="IC1" gate="G$1" pin="VOUT"/>
@@
 </segment>
 </net>
-<net name="GND" class="0">
+<net name="GND" class="1">
 <segment>
 <pinref part="GND1" gate="1" pin="GND"/>
@@
 <wire x1="58.42" y1="45.72" x2="58.42" y2="38.1" width="0.1524" layer="91"/>
 <pinref part="BAT_CON" gate="G$1" pin="2"/>
-<wire x1="20.32" y1="45.72" x2="22.86" y2="45.72" width="0.1524" layer="91"/>
-<wire x1="22.86" y1="45.72" x2="22.86" y2="38.1" width="0.1524" layer="91"/>
-<wire x1="22.86" y1="38.1" x2="35.56" y2="38.1" width="0.1524" layer="91"/>
+<wire x1="20.32" y1="38.1" x2="35.56" y2="38.1" width="0.1524" layer="91"/>
 <junction x="35.56" y="38.1"/>
 </segment>
@@
 </segment>
 <segment>
-<pinref part="U$1" gate="G$1" pin="VIN-"/>
+<pinref part="MT3608" gate="G$1" pin="VIN-"/>
 <wire x1="50.8" y1="-7.62" x2="48.26" y2="-7.62" width="0.1524" layer="91"/>
 <wire x1="48.26" y1="-7.62" x2="48.26" y2="-15.24" width="0.1524" layer="91"/>
@@
 <wire x1="68.58" y1="-15.24" x2="88.9" y2="-15.24" width="0.1524" layer="91"/>
 <wire x1="88.9" y1="-15.24" x2="88.9" y2="-7.62" width="0.1524" layer="91"/>
-<pinref part="U$1" gate="G$1" pin="VOUT-"/>
+<pinref part="MT3608" gate="G$1" pin="VOUT-"/>
 <wire x1="88.9" y1="-7.62" x2="86.36" y2="-7.62" width="0.1524" layer="91"/>
 <pinref part="GND8" gate="1" pin="GND"/>
@@
 </segment>
 </net>
-<net name="+12V" class="0">
+<net name="+12V" class="1">
 <segment>
 <pinref part="P+2" gate="1" pin="+12V"/>
@@
 </segment>
 <segment>
-<pinref part="U$1" gate="G$1" pin="VOUT+"/>
+<pinref part="MT3608" gate="G$1" pin="VOUT+"/>
 <wire x1="86.36" y1="0" x2="96.52" y2="0" width="0.1524" layer="91"/>
 <pinref part="P+8" gate="1" pin="+12V"/>
@@
 </segment>
 </net>
-<net name="N$1" class="0">
+<net name="N$1" class="1">
 <segment>
 <pinref part="SG1" gate="G$1" pin="-"/>
@@
 </segment>
 </net>
-<net name="MCU_VCC" class="0">
+<net name="MCU_VCC" class="1">
 <segment>
 <pinref part="U1" gate="G$1" pin="VCC"/>
@@
 </segment>
 </net>
-<net name="VPROG" class="0">
+<net name="VPROG" class="1">
 <segment>
 <pinref part="PROG/DEPL" gate="G$1" pin="1"/>
@@
 </segment>
 </net>
-<net name="N$2" class="0">
+<net name="N$2" class="2">
 <segment>
 <pinref part="NICHROME_WIRE" gate="-2" pin="KL"/>
@@
 </segment>
 </net>
+<net name="N$6" class="2">
+<segment>
+<pinref part="SWITCH" gate="G$1" pin="2"/>
+<wire x1="20.32" y1="50.8" x2="22.86" y2="50.8" width="0.1524" layer="91"/>
+<wire x1="22.86" y1="50.8" x2="22.86" y2="40.64" width="0.1524" layer="91"/>
+<pinref part="BAT_CON" gate="G$1" pin="1"/>
+<wire x1="22.86" y1="40.64" x2="20.32" y2="40.64" width="0.1524" layer="91"/>
+</segment>
+</net>
